Commit message: Change POs implementation

File: model/hopper.urdf (robot description, URDF)
Before this commit: robot hopper, 13 links, 12 joints
Joints:
- joint leg_joint: limit lower=-2.2 upper=0.5 effort=50 velocity=30 -> lower=-0.5 upper=2.2 effort=50 velocity=30
- joint thigh_joint: limit lower=-0.50000 upper=1.4 effort=50 velocity=30 -> lower=-1.4 upper=0.5 effort=50 velocity=30

Commit message: Change POs values and robot joint max/min values

File: model/hopper.urdf (robot description, URDF)
Before this commit: robot hopper, 13 links, 12 joints
Joints:
- joint leg_joint: limit lower=-0.5 upper=2.2 effort=50 velocity=30 -> lower=-2.2 upper=0.5 effort=50 velocity=30
- joint thigh_joint: limit lower=-1.4 upper=0.5 effort=50 velocity=30 -> lower=-0.5 upper=1.4 effort=50 velocity=30

Commit message: Hard code almost jump

File: model/hopper.urdf (robot description, URDF)
Before this commit: robot hopper, 13 links, 12 joints
Joints:
- joint leg_joint: limit lower=-2.2 upper=0.5 effort=50 velocity=30 -> lower=-0.5 upper=2.2 effort=50 velocity=30
- joint thigh_joint: limit lower=-0.5 upper=1.4 effort=50 velocity=30 -> lower=-1.4 upper=0.5 effort=50 velocity=30
